Commit message: added a base_footprint would prove useful when setting up navigation

File: slambot_description/urdf/slambot.xacro (robot description, xacro)
@@ -6,4 +6,5 @@
 <xacro:include filename="$(find slambot_description)/gazebo/slambot_physics.gazebo" />
 <xacro:include filename="$(find slambot_description)/gazebo/slambot_plugins.gazebo" />
+<link name="base_footprint"/>
 <link name="base_link">
   <inertial>
@@ -106,4 +107,8 @@
   </collision>
 </link>
+<joint name="base_joint" type="fixed">
+  <parent link="base_footprint"/>
+  <child link="base_link"/>
+</joint>
 <joint name="motor_right" type="continuous">
   <origin xyz="0.03275 -0.0722 0.033" rpy="0 0 0"/>
